File: Hardware/_autosave-Hardware.kicad_pcb (KiCad board)
At the start: 2 copper layers, 15 parts, among them J1 Conn_01x02, J2 Conn_01x04, J3 Conn_01x03, J4 Conn_01x02, J5 Conn_01x06, J6 Conn_01x08, U1 ESP32-WROOM-32

Commit message: Routing was done
Parts:
- moved J2 85.6 mm to (85.1, 121.9), turned to 90 degrees
- moved J4 68.5 mm to (85.1, 88.9), turned to 180 degrees
- moved R3 62.8 mm to (93.5, 114.3)
- moved R2 59.1 mm to (93.5, 111.8)
- moved R1 49.9 mm to (139.7, 90.2), turned to 90 degrees
- moved R4 49.1 mm to (107.2, 121.4), turned to 90 degrees
- moved C1 33.0 mm to (136.1, 84.3), turned to 180 degrees
- moved R5 32.2 mm to (115.8, 121.4), turned to 90 degrees
- moved C3 27.3 mm to (136.1, 92.9), turned to 180 degrees
- moved C2 26.9 mm to (136.1, 101.6), turned to 180 degrees
- moved J3 26.2 mm to (134.6, 111.8)
- moved J1 12.4 mm to (134.6, 124.5)
- moved J6 11.4 mm to (85.1, 114.3)
- moved J5 4.26 mm to (115.6, 129.5)
Routing:
- net Net-(C1-Pad1): track 0.00 -> 50.2 mm, vias 0 -> 2
- net /IO23: track 0.00 -> 47.5 mm, vias 0 -> 2
- net GND: track 0.00 -> 37.1 mm, vias 0 -> 3
- net /SDI: track 0.00 -> 34.2 mm, vias 0 -> 2
- net Net-(J2-Pad4): track 0.00 -> 25.6 mm, vias 0 -> 3
- net /SDO: track 0.00 -> 24.2 mm, vias 0 -> 1
- net /IO35: track 0.00 -> 21.2 mm
- net /IO33: track 0.00 -> 20.5 mm
- net Net-(J2-Pad3): track 0.00 -> 20.4 mm
- net /RXD: track 0.00 -> 20.3 mm
- net /IO27: track 0.00 -> 19.6 mm
- net /IO25: track 0.00 -> 19.6 mm, vias 0 -> 2
- net /TXD: track 0.00 -> 19.2 mm
- net /Boot_Option: track 0.00 -> 19.2 mm
- net /IO34: track 0.00 -> 19.0 mm, vias 0 -> 2
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- added copper zone on B.Cu, net /VDD33
- added copper zone on F.Cu, net /VDD33
- added copper zone on B.Cu, net GND
