File: Hardware/Hardware.kicad_pcb (KiCad board)
At the start: 2 copper layers, 18 parts, among them J1 Conn_01x02, J2 Conn_01x04, J3 Conn_01x03, J4 Conn_01x02, J5 Conn_01x06, J6 Conn_01x08, J7 Conn_01x03, U1 ESP32-WROOM-32

Commit message: A board was bought. Yayyyyy!
Other:
- board outline added: 66 x 57.1 mm
- board text added: "ESP32_REV_A"

Commit message: layout reworking
Parts:
- removed J5: Conn_01x06, Connector_PinHeader_2.54mm:PinHeader_1x06_P2.54mm_Vertical
- removed J6: Conn_01x08, Connector_PinHeader_2.54mm:PinHeader_1x08_P2.54mm_Vertical
- added D1: LED, LED_SMD:LED_0805_2012Metric_Castellated, F.Cu at (151.1, 113.0)
- J3: value Conn_01x03 -> Conn_01x06; footprint Connector_PinHeader_2.54mm:PinHeader_1x03_P2.54mm_Vertical -> Connector_PinHeader_2.54mm:PinHeader_1x06_P2.54mm_Vertical
- moved J3 11.9 mm to (146.4, 113.9)
Connections:
- C1 pad 1: Net-(C1-Pad1) -> /EN
- J3 pad 1: /TXD -> GND
- J3 pad 2: /RXD -> /EN
- J3 pad 3: GND -> (no net)
- R1 pad 2: Net-(C1-Pad1) -> /EN
- U1 pad 10: /IO25 -> (no net)
- U1 pad 11: /IO26 -> (no net)
- U1 pad 12: /IO27 -> (no net)
- U1 pad 17: /SHD -> (no net)
- U1 pad 18: /SWP -> (no net)
- U1 pad 19: /SCS -> (no net)
- U1 pad 20: /SCK -> (no net)
- U1 pad 21: /SDO -> (no net)
- U1 pad 22: /SDI -> (no net)
- U1 pad 3: Net-(C1-Pad1) -> /EN
- U1 pad 37: /IO23 -> (no net)
- U1 pad 6: /IO34 -> (no net)
- U1 pad 7: /IO35 -> (no net)
- U1 pad 8: /IO32 -> (no net)
Routing:
- net (no net): track 0.00 -> 74.0 mm, vias 0 -> 1
- net Net-(C1-Pad1): track 51.3 -> 0.00 mm, vias 2 -> 0
- net /EN: track 0.00 -> 51.3 mm, vias 0 -> 2
- net /IO23: track 47.5 -> 0.00 mm, vias 2 -> 0
- net /SDI: track 34.2 -> 0.00 mm, vias 2 -> 0
- net GND: track 78.8 -> 45.5 mm, vias 9 -> 6
- net /SDO: track 24.2 -> 0.00 mm, vias 1 -> 0
- net /IO35: track 21.2 -> 0.00 mm
- net /IO33: track 20.5 -> 0.00 mm
- net /IO27: track 19.6 -> 0.00 mm
- net /IO25: track 19.6 -> 0.00 mm, vias 2 -> 0
- net /IO34: track 19.0 -> 0.00 mm, vias 2 -> 0
- net /IO32: track 18.6 -> 0.00 mm, vias 2 -> 0
- net /IO26: track 17.4 -> 0.00 mm, vias 2 -> 0
- net /SCS: track 16.9 -> 0.00 mm
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Other:
- board text removed: "IO23"
- board text removed: "IO25"
- board text removed: "IO26"
- board text removed: "IO27"
- board text removed: "IO32"
- board text removed: "IO33"
- board text removed: "IO34"
- board text removed: "IO35"

Commit message: Layout updates
Parts:
- removed C3: 0.1uF, Capacitor_SMD:C_0805_2012Metric
- moved D1 52.7 mm to (98.8, 107.3)
- moved C2 40.2 mm to (95.9, 101.2), turned to 90 degrees
- moved J3 23.3 mm to (127.0, 101.0)
- moved C1 19.1 mm to (131.4, 102.9), turned to 0 degrees
- moved R1 19.0 mm to (131.4, 107.3), turned to 180 degrees
- moved J4 15.1 mm to (90.8, 102.9)
- moved J1 9.16 mm to (127.0, 119.4), turned to 270 degrees
Routing:
- net (no net): track 74.0 -> 0.00 mm, vias 1 -> 0
- net GND: track 45.5 -> 26.3 mm
- net /EN: track 51.3 -> 35.0 mm, vias 2 -> 1
- net /RXD: track 20.3 -> 10.7 mm
- net Net-(J2-Pad4): track 21.0 -> 30.6 mm
- net /Boot_Option: track 19.2 -> 12.8 mm
- net /TXD: track 19.2 -> 13.9 mm, vias 0 -> 2
- net /IO33: track 0.00 -> 3.16 mm
- net Net-(U1-Pad20): track 2.54 -> 0.00 mm
- net /VDD33: track 2.00 -> 0.47 mm
Other:
- board text removed: "SERIAL"

Commit message: Board revision
Parts:
- moved J7 15.7 mm to (87.9, 113.8), turned to 180 degrees
- moved J2 9.51 mm to (94.5, 120.7)
- moved H2 9.34 mm to (133.1, 125.5)
Routing:
- net /MTMS: track 46.3 -> 18.6 mm, vias 1 -> 0
- net Net-(J2-Pad4): track 30.6 -> 16.9 mm, vias 3 -> 0
- net Net-(J2-Pad3): track 21.5 -> 10.4 mm
- net GND: track 26.3 -> 16.1 mm, vias 6 -> 7
- net /MTDO: track 9.07 -> 5.19 mm
- net Net-(J2-Pad1): track 13.4 -> 11.9 mm
- net Net-(J2-Pad2): track 9.72 -> 10.5 mm
Other:
- board outline removed
- board text removed: "JTAG"

Commit message: board revising
Parts:
- moved H1 10.5 mm to (83.8, 121.9)
- moved H2 3.87 mm to (134.6, 121.9)
Other:
- board outline added: 58.4 x 30.5 mm
- board text added: "ESP32_REV_B"
- board text removed: "ESP32_REV_A"
Changed lines of the file:
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@@
     (pad_to_mask_clearance 0)
     (aux_axis_origin 0 0)
-    (visible_elements 7FFFF7FF)
+    (visible_elements 7FFFFFFF)
     (pcbplotparams
       (layerselection 0x010fc_ffffffff)
@@
     (tags resistor)
     (attr smd)
-    (fp_text reference R3 (at 0 -1.65) (layer F.SilkS)
+    (fp_text reference R3 (at 0 1.905) (layer F.SilkS)
       (effects (font (size 1 1) (thickness 0.15)))
     )
@@
     )
   )
-  (module MountingHole:MountingHole_2.1mm (layer F.Cu)
-    (at 133.096 125.476)
+  (module MountingHole:MountingHole_2.1mm locked (layer F.Cu)
+    (at 134.62 121.92)
     (descr "Mounting Hole 2.1mm, no annular")
     (tags "mounting hole 2.1mm no annular")
@@
   )
   (module MountingHole:MountingHole_2.1mm locked (layer F.Cu)
-    (at 81.28 132.08)
+    (at 83.82 121.92)
     (descr "Mounting Hole 2.1mm, no annular")
     (tags "mounting hole 2.1mm no annular")
@@
     )
   )
-  (dimension 66.04 (width 0.15) (layer Dwgs.User)
-    (gr_text "66.040 mm" (at 110.49 72.36) (layer Dwgs.User)
-      (effects (font (size 1 1) (thickness 0.15)))
-    )
-    (feature1 (pts (xy 143.51 78.74) (xy 143.51 73.073579)))
-    (feature2 (pts (xy 77.47 78.74) (xy 77.47 73.073579)))
-    (crossbar (pts (xy 77.47 73.66) (xy 143.51 73.66)))
-    (arrow1a (pts (xy 143.51 73.66) (xy 142.383496 74.246421)))
-    (arrow1b (pts (xy 143.51 73.66) (xy 142.383496 73.073579)))
-    (arrow2a (pts (xy 77.47 73.66) (xy 78.596504 74.246421)))
-    (arrow2b (pts (xy 77.47 73.66) (xy 78.596504 73.073579)))
-  )
-  (gr_line (start 143.51 78.74) (end 77.47 78.74) (layer Dwgs.User) (width 0.15))
+  (gr_line (start 138.43 96.52) (end 138.43 127) (layer Edge.Cuts) (width 0.1))
+  (gr_line (start 80.01 96.52) (end 138.43 96.52) (layer Edge.Cuts) (width 0.1))
+  (gr_line (start 80.01 127) (end 80.01 96.52) (layer Edge.Cuts) (width 0.1))
+  (gr_line (start 138.43 127) (end 80.01 127) (layer Edge.Cuts) (width 0.1))
   (gr_line (start 77.47 135.89) (end 143.51 135.89) (layer Dwgs.User) (width 0.15))
-  (gr_text ESP32_REV_A (at 132.08 134.62) (layer F.SilkS)
+  (gr_text ESP32_REV_B (at 82.55 102.87 -90) (layer F.SilkS)
     (effects (font (size 1 1) (thickness 0.15)))
-  )
-  (dimension 57.15 (width 0.15) (layer Dwgs.User)
-    (gr_text "57.150 mm" (at 72.36 107.315 90) (layer Dwgs.User)
-      (effects (font (size 1 1) (thickness 0.15)))
-    )
-    (feature1 (pts (xy 77.47 78.74) (xy 73.073579 78.74)))
-    (feature2 (pts (xy 77.47 135.89) (xy 73.073579 135.89)))
-    (crossbar (pts (xy 73.66 135.89) (xy 73.66 78.74)))
-    (arrow1a (pts (xy 73.66 78.74) (xy 74.246421 79.866504)))
-    (arrow1b (pts (xy 73.66 78.74) (xy 73.073579 79.866504)))
-    (arrow2a (pts (xy 73.66 135.89) (xy 74.246421 134.763496)))
-    (arrow2b (pts (xy 73.66 135.89) (xy 73.073579 134.763496)))
   )
   (gr_text BOOT (at 124.5235 121.9835) (layer F.SilkS)
@@
     (effects (font (size 1 1) (thickness 0.15)))
   )
-  (gr_text Motor (at 87.63 132.08) (layer F.SilkS)
+  (gr_text Motor (at 85.09 109.22 270) (layer F.SilkS)
     (effects (font (size 1 1) (thickness 0.15)))
   )
-  (gr_line (start 77.47 78.74) (end 77.47 135.89) (layer Dwgs.User) (width 0.15))
   (via (at 109.855 105.41) (size 0.8) (drill 0.4) (layers F.Cu B.Cu) (net 1))
   (segment (start 109.855 105.41) (end 109.855 104.775) (width 0.25) (layer F.Cu) (net 1))
@@
     (connect_pads (clearance 0.508))
     (min_thickness 0.254)
-    (fill yes (arc_segments 32) (thermal_gap 0.508) (thermal_bridge_width 0.508))
+    (fill (arc_segments 32) (thermal_gap 0.508) (thermal_bridge_width 0.508))
     (polygon
       (pts
         (xy 95.25 96.52) (xy 104.14 96.52) (xy 104.14 113.03) (xy 118.11 113.03) (xy 118.11 96.52)
-        (xy 127 96.52) (xy 143.51 96.52) (xy 143.51 135.89) (xy 77.47 135.89) (xy 77.47 96.52)
+        (xy 127 96.52) (xy 138.43 96.52) (xy 138.43 127) (xy 80.01 127) (xy 80.01 96.52)
       )
     )
@@
     (connect_pads (clearance 0.508))
     (min_thickness 0.254)
-    (fill yes (arc_segments 32) (thermal_gap 0.508) (thermal_bridge_width 0.508))
+    (fill (arc_segments 32) (thermal_gap 0.508) (thermal_bridge_width 0.508))
     (polygon
       (pts
-        (xy 95.25 96.52) (xy 127 96.52) (xy 143.51 96.52) (xy 143.51 135.89) (xy 77.47 135.89)
-        (xy 77.47 96.52)
+        (xy 95.25 96.52) (xy 127 96.52) (xy 138.43 96.52) (xy 138.43 127) (xy 80.01 127)
+        (xy 80.01 96.52)
       )
     )
